Commit message: launch multi robot -gz sim- done

File: src/gazebo_simulation/worlds/slide_1.world.xacro (robot description, xacro)
@@ -1,4 +1,31 @@
-<sdf version='1.6'>
+<?xml version="1.0"?>
+<sdf version="1.6" xmlns:xacro="http://www.ros.org/wiki/xacro">
   <world name='ur_world_1'>
+    <plugin
+      filename="gz-sim-physics-system"
+      name="gz::sim::systems::Physics">
+    </plugin>
+    <plugin
+      filename="gz-sim-user-commands-system"
+      name="gz::sim::systems::UserCommands">
+    </plugin>
+    <plugin
+      filename="gz-sim-navsat-system"
+      name="gz::sim::systems::NavSat">
+    </plugin>
+    <xacro:unless value="$(arg headless)">
+      <plugin
+        filename="gz-sim-scene-broadcaster-system"
+        name="gz::sim::systems::SceneBroadcaster">
+      </plugin>
+    </xacro:unless>
+    <plugin
+      filename="gz-sim-sensors-system"
+      name="gz::sim::systems::Sensors">
+    </plugin>
+    <plugin
+      filename="gz-sim-imu-system"
+      name="gz::sim::systems::Imu">
+    </plugin>
     <light name='sun' type='directional'>
       <cast_shadows>0</cast_shadows>
@@ -27,5 +54,5 @@
             <contact>
               <collide_bitmask>65535</collide_bitmask>
-              <ode/>
+              <ode />
             </contact>
             <friction>
@@ -35,8 +62,8 @@
               </ode>
               <torsional>
-                <ode/>
-              </torsional>
-            </friction>
-            <bounce/>
+                <ode />
+              </torsional>
+            </friction>
+            <bounce />
           </surface>
           <max_contacts>10</max_contacts>
@@ -64,5 +91,5 @@
     <gravity>0 0 -9.8</gravity>
     <magnetic_field>6e-06 2.3e-05 -4.2e-05</magnetic_field>
-    <atmosphere type='adiabatic'/>
+    <atmosphere type='adiabatic' />
     <physics name='default_physics' default='0' type='ode'>
       <max_step_size>0.001</max_step_size>
@@ -78,5 +105,5 @@
       <device>default</device>
     </audio>
-    <wind/>
+    <wind />
     <spherical_coordinates>
       <surface_model>EARTH_WGS84</surface_model>
@@ -99,12 +126,12 @@
           <surface>
             <contact>
-              <ode/>
-            </contact>
-            <bounce/>
-            <friction>
-              <torsional>
-                <ode/>
-              </torsional>
-              <ode/>
+              <ode />
+            </contact>
+            <bounce />
+            <friction>
+              <torsional>
+                <ode />
+              </torsional>
+              <ode />
             </friction>
           </surface>
@@ -163,12 +190,12 @@
           <surface>
             <contact>
-              <ode/>
-            </contact>
-            <bounce/>
-            <friction>
-              <torsional>
-                <ode/>
-              </torsional>
-              <ode/>
+              <ode />
+            </contact>
+            <bounce />
+            <friction>
+              <torsional>
+                <ode />
+              </torsional>
+              <ode />
             </friction>
           </surface>
@@ -202,12 +229,12 @@
           <surface>
             <contact>
-              <ode/>
-            </contact>
-            <bounce/>
-            <friction>
-              <torsional>
-                <ode/>
-              </torsional>
-              <ode/>
+              <ode />
+            </contact>
+            <bounce />
+            <friction>
+              <torsional>
+                <ode />
+              </torsional>
+              <ode />
             </friction>
           </surface>
@@ -241,12 +268,12 @@
           <surface>
             <contact>
-              <ode/>
-            </contact>
-            <bounce/>
-            <friction>
-              <torsional>
-                <ode/>
-              </torsional>
-              <ode/>
+              <ode />
+            </contact>
+            <bounce />
+            <friction>
+              <torsional>
+                <ode />
+              </torsional>
+              <ode />
             </friction>
           </surface>
@@ -280,12 +307,12 @@
           <surface>
             <contact>
-              <ode/>
-            </contact>
-            <bounce/>
-            <friction>
-              <torsional>
-                <ode/>
-              </torsional>
-              <ode/>
+              <ode />
+            </contact>
+            <bounce />
+            <friction>
+              <torsional>
+                <ode />
+              </torsional>
+              <ode />
             </friction>
           </surface>
@@ -319,12 +346,12 @@
           <surface>
             <contact>
-              <ode/>
-            </contact>
-            <bounce/>
-            <friction>
-              <torsional>
-                <ode/>
-              </torsional>
-              <ode/>
+              <ode />
+            </contact>
+            <bounce />
+            <friction>
+              <torsional>
+                <ode />
+              </torsional>
+              <ode />
             </friction>
           </surface>
@@ -358,12 +385,12 @@
           <surface>
             <contact>
-              <ode/>
-            </contact>
-            <bounce/>
-            <friction>
-              <torsional>
-                <ode/>
-              </torsional>
-              <ode/>
+              <ode />
+            </contact>
+            <bounce />
+            <friction>
+              <torsional>
+                <ode />
+              </torsional>
+              <ode />
             </friction>
           </surface>
@@ -397,12 +424,12 @@
           <surface>
             <contact>
-              <ode/>
-            </contact>
-            <bounce/>
-            <friction>
-              <torsional>
-                <ode/>
-              </torsional>
-              <ode/>
+              <ode />
+            </contact>
+            <bounce />
+            <friction>
+              <torsional>
+                <ode />
+              </torsional>
+              <ode />
             </friction>
           </surface>
@@ -436,12 +463,12 @@
           <surface>
             <contact>
-              <ode/>
-            </contact>
-            <bounce/>
-            <friction>
-              <torsional>
-                <ode/>
-              </torsional>
-              <ode/>
+              <ode />
+            </contact>
+            <bounce />
+            <friction>
+              <torsional>
+                <ode />
+              </torsional>
+              <ode />
             </friction>
           </surface>
@@ -475,12 +502,12 @@
           <surface>
             <contact>
-              <ode/>
-            </contact>
-            <bounce/>
-            <friction>
-              <torsional>
-                <ode/>
-              </torsional>
-              <ode/>
+              <ode />
+            </contact>
+            <bounce />
+            <friction>
+              <torsional>
+                <ode />
+              </torsional>
+              <ode />
             </friction>
           </surface>
@@ -514,12 +541,12 @@
           <surface>
             <contact>
-              <ode/>
-            </contact>
-            <bounce/>
-            <friction>
-              <torsional>
-                <ode/>
-              </torsional>
-              <ode/>
+              <ode />
+            </contact>
+            <bounce />
+            <friction>
+              <torsional>
+                <ode />
+              </torsional>
+              <ode />
             </friction>
           </surface>
@@ -540,12 +567,12 @@
           <surface>
             <contact>
-              <ode/>
-            </contact>
-            <bounce/>
-            <friction>
-              <torsional>
-                <ode/>
-              </torsional>
-              <ode/>
+              <ode />
+            </contact>
+            <bounce />
+            <friction>
+              <torsional>
+                <ode />
+              </torsional>
+              <ode />
             </friction>
           </surface>
@@ -604,12 +631,12 @@
           <surface>
             <contact>
-              <ode/>
-            </contact>
-            <bounce/>
-            <friction>
-              <torsional>
-                <ode/>
-              </torsional>
-              <ode/>
+              <ode />
+            </contact>
+            <bounce />
+            <friction>
+              <torsional>
+                <ode />
+              </torsional>
+              <ode />
             </friction>
           </surface>
@@ -643,12 +670,12 @@
           <surface>
             <contact>
-              <ode/>
-            </contact>
-            <bounce/>
-            <friction>
-              <torsional>
-                <ode/>
-              </torsional>
-              <ode/>
+              <ode />
+            </contact>
+            <bounce />
+            <friction>
+              <torsional>
+                <ode />
+              </torsional>
+              <ode />
             </friction>
           </surface>
@@ -682,12 +709,12 @@
           <surface>
             <contact>
-              <ode/>
-            </contact>
-            <bounce/>
-            <friction>
-              <torsional>
-                <ode/>
-              </torsional>
-              <ode/>
+              <ode />
+            </contact>
+            <bounce />
+            <friction>
+              <torsional>
+                <ode />
+              </torsional>
+              <ode />
             </friction>
           </surface>
@@ -721,12 +748,12 @@
           <surface>
             <contact>
-              <ode/>
-            </contact>
-            <bounce/>
-            <friction>
-              <torsional>
-                <ode/>
-              </torsional>
-              <ode/>
+              <ode />
+            </contact>
+            <bounce />
+            <friction>
+              <torsional>
+                <ode />
+              </torsional>
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
File: src/robot_description/urdf/uvc_robot_gazebo.xacro (robot description, xacro)
@@ -37,11 +37,6 @@
         </plugin>
     </gazebo>
+    <!-- sensors ===============================================  -->
     <!-- velodyne_laserscan ===============================================  -->
-    <!-- <gazebo>
-        <plugin
-            filename="libgz-sim-sensors-system"
-            name="gz::sim::systems::Sensors">
-        </plugin>
-    </gazebo> -->
     <gazebo reference="velodyne_laserscan">
         <sensor type="gpu_lidar" name="velodyne_laserscan">

File: src/robot_description/urdf/uvc_robot_m_gazebo.xacro (robot description, xacro)
@@ -1,6 +1,6 @@
 <?xml version="1.0"?>
 <robot name="uvc_robot" xmlns:xacro="http://www.ros.org/wiki/xacro">
-    <xacro:arg name="robot_name" default="" />
-    <xacro:property name="robot_name" value="$(arg robot_name)" />
+    <xacro:arg name="namespace" default="" />
+    <xacro:property name="namespace" value="$(arg namespace)" />
     <gazebo reference="base_link">
         <material>Gazebo/Orange</material>
@@ -24,9 +24,9 @@
             <wheel_radius>0.0775</wheel_radius>
             <odom_publish_frequency>20</odom_publish_frequency>
-            <topic>${robot_name}/cmd_vel</topic>
-            <odom_topic>${robot_name}/odom</odom_topic>
-            <tf_topic>tf</tf_topic>
-            <frame_id>${robot_name}/odom</frame_id>
-            <child_frame_id>${robot_name}/base_link</child_frame_id>
+            <topic>${namespace}/cmd_vel</topic>
+            <odom_topic>${namespace}/odom</odom_topic>
+            <tf_topic>${namespace}/tf</tf_topic>
+            <frame_id>${namespace}/odom</frame_id>
+            <child_frame_id>${namespace}/base_link</child_frame_id>
             <max_linear_acceleration>1</max_linear_acceleration>
             <min_linear_acceleration>-1</min_linear_acceleration>
@@ -39,12 +39,6 @@
         </plugin>
     </gazebo>
+    <!-- sensors ===============================================  -->
     <!-- velodyne_laserscan ===============================================  -->
-    <!--
-    <gazebo>
-        <plugin
-            filename="libgz-sim-sensors-system"
-            name="gz::sim::systems::Sensors">
-        </plugin>
-    </gazebo> -->
     <gazebo reference="velodyne_laserscan">
         <sensor type="gpu_lidar" name="velodyne_laserscan">
@@ -53,6 +47,6 @@
             <visualize>false</visualize>
             <update_rate>5</update_rate>
-            <topic>${robot_name}/velodyne_laserscan</topic>
-            <gz_frame_id>${robot_name}/velodyne_laserscan</gz_frame_id>
+            <topic>${namespace}/velodyne_laserscan</topic>
+            <gz_frame_id>${namespace}/velodyne_laserscan</gz_frame_id>
             <ray>
                 <scan>
@@ -75,8 +69,4 @@
                 </noise>
             </ray>
-            <!-- <plugin
-                filename="libgz-sim-sensors-system"
-                name="gz::sim::systems::Sensors">
-            </plugin> -->
         </sensor>
     </gazebo>
@@ -87,5 +77,5 @@
             <visualize>true</visualize>
             <update_rate>2.0</update_rate>
-            <topic>${robot_name}/usb_cam</topic>
+            <topic>${namespace}/usb_cam</topic>
             <camera>
                 <horizontal_fov>1.047198</horizontal_fov>
